File: adafruit-cp2104-friend-adapter/project.kicad_pcb (KiCad board)
At the start: 2 copper layers, 34.6 x 30.4 mm, 15 parts, among them J1 Conn_02x09_Odd_Even, J2 Conn_02x09_Odd_Even, J3 Conn_01x08_Female, J4 Conn_01x08_Female, Q1 S8050, Q2 S8050, U1 AMS1117

Commit message: Fixes to beta1 versions and added rws
Parts:
- removed Q2: S8050, Package_TO_SOT_SMD:SOT-23
- removed the R1 at (143.1, 109.6)
- removed R2: 10k, Resistor_SMD:R_1206_3216Metric_Pad1.30x1.75mm_HandSolder
- added J5: +/- rail, Connector_PinHeader_2.54mm:PinHeader_2x06_P2.54mm_Vertical, B.Cu at (149.7, 91.0)
- added J6: Conn_01x03, Connector_PinHeader_2.54mm:PinHeader_1x03_P2.54mm_Vertical, B.Cu at (132.6, 114.6)
- C3: value 22uF -> 100nF
- Q1: value S8050 -> MUN5214DW1; footprint Package_TO_SOT_SMD:SOT-23 -> Package_TO_SOT_SMD:SOT-363_SC-70-6
- U1: value AMS1117 -> AZ1117
- moved C1 18.1 mm to (140.2, 108.3)
- moved C3 10.6 mm to (146.0, 108.3)
- moved U1 10.2 mm to (143.1, 101.0), turned to 90 degrees
- moved Q1 8.95 mm to (143.1, 108.5)
- moved REF** 8.48 mm to (143.5, 95.6)
- moved C2 7.98 mm to (143.2, 94.3), turned to 180 degrees
- moved R1 2.75 mm to (142.9, 114.9)
- moved D1 2.40 mm to (143.0, 112.3)
- renumbered R3 to R1
Connections:
- C1 pad 1: /+5v -> /+5v-out
- J2 pad 13: /RXD -> /ESP-RX
- J2 pad 15: /TXD -> /ESP-TX
- J3 pad 1: /+5v -> /+5v-in
- J4 pad 5: /TXD -> /ESP-RX
- J4 pad 6: /RXD -> /ESP-TX
- Q1 pad 1: /RTS -> /DTR
- Q1 pad 2: Net-(Q1-Pad2) -> /RTS
- R1 pad 2: /+5v -> /+5v-out
- U1 pad 3: /+5v -> /+5v-out
Routing:
- net /+5v-out: track 0.00 -> 41.0 mm, vias 0 -> 2
- net /+5v: track 30.2 -> 0.00 mm
- net /TXD: track 20.7 -> 0.00 mm
- net /VDD: track 19.8 -> 35.9 mm
- net /ESP-RX: track 0.00 -> 15.9 mm
- net /ESP-TX: track 0.00 -> 15.8 mm
- net /RXD: track 13.6 -> 0.00 mm
- net Net-(Q1-Pad2): track 11.3 -> 0.00 mm, vias 2 -> 0
- net /EN: track 18.0 -> 28.2 mm
- net /GND: track 67.6 -> 74.6 mm, vias 3 -> 1
- net /IO0: track 12.8 -> 19.6 mm, vias 0 -> 1
- net /+5v-in: track 0.00 -> 4.50 mm
- net Net-(Q2-Pad2): track 3.04 -> 0.00 mm
- net /RTS: track 12.6 -> 15.1 mm, vias 0 -> 1
- net /IO15: track 0.94 -> 0.00 mm
Other:
- board text added: "+3.3v"
- board text added: "12|13"
- board text added: "17|16"
- board text added: "18|5"
- board text added: "21|19"
- board text added: "25|26"
- board text added: "27|14"
- board text added: "2|15"
- board text added: "2|3"
- board text added: "32|33"
- board text added: "34|35"
- board text added: "3v|GN"
- board text added: "4|0"
- board text added: "CMD|CLK"
- board text added: "ESP32 CP2104 adapter (c) 2021 dushin.net v0.1.0-beta2"
- board text added: "GN|22"
- board text added: "RX|23"
- board text added: "SD0|SD1"
- board text added: "SVP|SVN"
- board text added: "TX|EN"
- board text added: "off"
- board text added: "on"
- board text removed: "ESP32 CP2104 adapter (c) 2021 dushin.net v0.1.0-beta1"
- board text removed: "Top"

Commit message: Fixup and wiring of rws
Parts:
- moved J5 0.30 mm to (149.7, 90.7)
Other:
- board text added: "02|03"
- board text added: "02|15"
- board text added: "04|00"
- board text added: "18|05"
- board text removed: "18|5"
- board text removed: "2|15"
- board text removed: "2|3"
- board text removed: "4|0"
Changed lines of the file:
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@@
     (thickness 1.6)
     (drawings 41)
-    (tracks 103)
+    (tracks 109)
     (zones 0)
     (modules 14)
@@
     (0 F.Cu signal)
     (31 B.Cu signal)
-    (32 B.Adhes user hide)
+    (32 B.Adhes user)
     (33 F.Adhes user)
-    (34 B.Paste user hide)
+    (34 B.Paste user)
     (35 F.Paste user)
-    (36 B.SilkS user hide)
+    (36 B.SilkS user)
     (37 F.SilkS user)
-    (38 B.Mask user hide)
+    (38 B.Mask user)
     (39 F.Mask user)
     (40 Dwgs.User user)
@@
     (44 Edge.Cuts user)
     (45 Margin user)
-    (46 B.CrtYd user hide)
+    (46 B.CrtYd user)
     (47 F.CrtYd user)
-    (48 B.Fab user hide)
+    (48 B.Fab user)
     (49 F.Fab user)
   )
@@
   )
   (module Connector_PinHeader_2.54mm:PinHeader_2x06_P2.54mm_Vertical (layer B.Cu)
-    (at 149.7404 91.0016 90)
+    (at 149.7404 90.7016 90)
     (descr "Through hole straight pin header, 2x06, 2.54mm pitch, double rows")
     (tags "Through hole pin header THT 2x06 2.54mm double row")
@@
     (effects (font (size 0.5 0.5) (thickness 0.125)) (justify mirror))
   )
-  (gr_text 2|3 (at 133.2904 103.6516) (layer B.SilkS)
+  (gr_text 02|03 (at 133.2904 103.6516) (layer B.SilkS)
     (effects (font (size 0.5 0.5) (thickness 0.125)) (justify mirror))
   )
@@
     (effects (font (size 0.5 0.5) (thickness 0.125)) (justify mirror))
   )
-  (gr_text 2|15 (at 152.3904 108.7516) (layer B.SilkS)
-    (effects (font (size 0.5 0.5) (thickness 0.125)) (justify mirror))
-  )
-  (gr_text 4|0 (at 152.3404 106.2016) (layer B.SilkS)
+  (gr_text 02|15 (at 152.3904 108.7516) (layer B.SilkS)
+    (effects (font (size 0.5 0.5) (thickness 0.125)) (justify mirror))
+  )
+  (gr_text 04|00 (at 152.3404 106.2016) (layer B.SilkS)
     (effects (font (size 0.5 0.5) (thickness 0.125)) (justify mirror))
   )
@@
     (effects (font (size 0.5 0.5) (thickness 0.125)) (justify mirror))
   )
-  (gr_text 18|5 (at 152.3904 101.1016) (layer B.SilkS)
+  (gr_text 18|05 (at 152.3904 101.1016) (layer B.SilkS)
     (effects (font (size 0.5 0.5) (thickness 0.125)) (justify mirror))
   )
@@
   (segment (start 157.9372 88.392) (end 156.6672 89.662) (width 0.25) (layer F.Cu) (net 1))
   (segment (start 144.6104 94.1591) (end 144.7529 94.3016) (width 0.25) (layer F.Cu) (net 1))
-  (segment (start 152.4959 91.0016) (end 153.8355 89.662) (width 0.25) (layer F.Cu) (net 1))
-  (segment (start 137.0404 91.0016) (end 152.4959 91.0016) (width 0.25) (layer F.Cu) (net 1))
   (segment (start 144.6604 96.2316) (end 143.0904 97.8016) (width 0.25) (layer F.Cu) (net 1))
-  (segment (start 144.6604 91.0016) (end 144.6604 96.2316) (width 0.25) (layer F.Cu) (net 1))
   (segment (start 143.0904 97.8016) (end 143.0904 104.1016) (width 0.25) (layer F.Cu) (net 1))
+  (segment (start 152.7959 90.7016) (end 153.8355 89.662) (width 0.25) (layer F.Cu) (net 1))
+  (segment (start 137.0404 90.7016) (end 152.7959 90.7016) (width 0.25) (layer F.Cu) (net 1))
+  (segment (start 144.6604 90.7016) (end 144.6604 92.5216) (width 0.25) (layer F.Cu) (net 1))
+  (segment (start 144.7529 92.6141) (end 144.7529 94.3016) (width 0.25) (layer F.Cu) (net 1))
+  (segment (start 144.6604 92.5216) (end 144.7529 92.6141) (width 0.25) (layer F.Cu) (net 1))
+  (segment (start 144.7529 96.1391) (end 144.6604 96.2316) (width 0.25) (layer F.Cu) (net 1))
+  (segment (start 144.7529 94.3016) (end 144.7529 96.1391) (width 0.25) (layer F.Cu) (net 1))
   (segment (start 145.9779 109.7516) (end 146.0404 109.8141) (width 0.25) (layer F.Cu) (net 2))
   (segment (start 155.3972 90.932) (end 154.11 90.932) (width 0.25) (layer F.Cu) (net 2))
@@
   (segment (start 155.829 88.392) (end 156.762199 89.325199) (width 0.25) (layer B.Cu) (net 31))
   (segment (start 137.11 88.392) (end 137.0404 88.4616) (width 0.25) (layer B.Cu) (net 31))
-  (segment (start 155.3972 88.392) (end 137.11 88.392) (width 0.25) (layer B.Cu) (net 31))
   (segment (start 140.1904 106.6891) (end 146.0404 106.6891) (width 0.25) (layer F.Cu) (net 31))
   (segment (start 140.7904 104.1016) (end 140.7904 105.0016) (width 0.25) (layer F.Cu) (net 31))
@@
   (segment (start 139.6293 106.6891) (end 140.1904 106.6891) (width 0.25) (layer F.Cu) (net 31))
   (segment (start 136.7774 109.541) (end 139.6293 106.6891) (width 0.25) (layer F.Cu) (net 31))
-  (segment (start 137.0404 88.4616) (end 135.3804 88.4616) (width 0.25) (layer F.Cu) (net 31))
-  (segment (start 135.3804 88.4616) (end 134.4904 89.3516) (width 0.25) (layer F.Cu) (net 31))
-  (segment (start 134.4904 89.3516) (end 134.4904 92.5516) (width 0.25) (layer F.Cu) (net 31))
-  (segment (start 136.2404 94.3016) (end 141.6279 94.3016) (width 0.25) (layer F.Cu) (net 31))
-  (segment (start 134.4904 92.5516) (end 136.2404 94.3016) (width 0.25) (layer F.Cu) (net 31))
   (segment (start 140.7904 104.1016) (end 140.7904 102.6016) (width 0.25) (layer F.Cu) (net 31))
   (segment (start 140.7904 102.6016) (end 139.7404 101.5516) (width 0.25) (layer F.Cu) (net 31))
@@
   (segment (start 142.9904 112.2516) (end 139.488 112.2516) (width 0.25) (layer B.Cu) (net 31))
   (segment (start 155.3972 88.392) (end 156.0068 88.392) (width 0.25) (layer B.Cu) (net 31))
-  (segment (start 151.6404 99.8342) (end 149.5536 101.921) (width 0.25) (layer F.Cu) (net 50))
-  (segment (start 151.6404 95.1016) (end 151.6404 99.8342) (width 0.25) (layer F.Cu) (net 50))
-  (segment (start 154.5404 92.2016) (end 151.6404 95.1016) (width 0.25) (layer F.Cu) (net 50))
-  (segment (start 156.7004 92.2016) (end 154.5404 92.2016) (width 0.25) (layer F.Cu) (net 50))
-  (segment (start 157.9804 90.9216) (end 156.7004 92.2016) (width 0.25) (layer F.Cu) (net 50))
-  (segment (start 152.6404 101.3742) (end 149.5536 104.461) (width 0.25) (layer F.Cu) (net 51))
-  (segment (start 152.6404 96.3516) (end 152.6404 101.3742) (width 0.25) (layer F.Cu) (net 51))
-  (segment (start 154.2404 94.7516) (end 152.6404 96.3516) (width 0.25) (layer F.Cu) (net 51))
-  (segment (start 156.6904 94.7516) (end 154.2404 94.7516) (width 0.25) (layer F.Cu) (net 51))
-  (segment (start 157.9804 93.4616) (end 156.6904 94.7516) (width 0.25) (layer F.Cu) (net 51))
+  (segment (start 135.5304 88.1616) (end 149.7404 88.1616) (width 0.25) (layer F.Cu) (net 31))
+  (segment (start 134.4904 89.2016) (end 135.5304 88.1616) (width 0.25) (layer F.Cu) (net 31))
+  (segment (start 134.4904 92.5516) (end 134.4904 89.2016) (width 0.25) (layer F.Cu) (net 31))
+  (segment (start 136.2404 94.3016) (end 134.4904 92.5516) (width 0.25) (layer F.Cu) (net 31))
+  (segment (start 141.6279 94.3016) (end 136.2404 94.3016) (width 0.25) (layer F.Cu) (net 31))
+  (segment (start 149.7404 88.1616) (end 152.9004 88.1616) (width 0.25) (layer F.Cu) (net 31))
+  (segment (start 153.1204 88.3816) (end 155.4404 88.3816) (width 0.25) (layer F.Cu) (net 31))
+  (segment (start 152.9004 88.1616) (end 153.1204 88.3816) (width 0.25) (layer F.Cu) (net 31))
   (segment (start 143.0904 108.991598) (end 143.0904 109.4516) (width 0.25) (layer F.Cu) (net 41))
   (segment (start 143.7404 108.341598) (end 143.0904 108.991598) (width 0.25) (layer F.Cu) (net 41))
@@
   (segment (start 136.758 114.6016) (end 136.7774 114.621) (width 0.25) (layer F.Cu) (net 48))
   (segment (start 132.2904 114.6016) (end 136.758 114.6016) (width 0.25) (layer F.Cu) (net 48))
+  (segment (start 151.6404 99.8342) (end 149.5536 101.921) (width 0.25) (layer F.Cu) (net 50))
+  (segment (start 151.6404 95.1016) (end 151.6404 99.8342) (width 0.25) (layer F.Cu) (net 50))
+  (segment (start 154.5404 92.2016) (end 151.6404 95.1016) (width 0.25) (layer F.Cu) (net 50))
+  (segment (start 156.7004 92.2016) (end 154.5404 92.2016) (width 0.25) (layer F.Cu) (net 50))
+  (segment (start 157.9804 90.9216) (end 156.7004 92.2016) (width 0.25) (layer F.Cu) (net 50))
+  (segment (start 152.6404 101.3742) (end 149.5536 104.461) (width 0.25) (layer F.Cu) (net 51))
+  (segment (start 152.6404 96.3516) (end 152.6404 101.3742) (width 0.25) (layer F.Cu) (net 51))
+  (segment (start 154.2404 94.7516) (end 152.6404 96.3516) (width 0.25) (layer F.Cu) (net 51))
+  (segment (start 156.6904 94.7516) (end 154.2404 94.7516) (width 0.25) (layer F.Cu) (net 51))
+  (segment (start 157.9804 93.4616) (end 156.6904 94.7516) (width 0.25) (layer F.Cu) (net 51))
 )

Commit message: Set version to v0.1.0
Other:
- board text added: "ESP32 CP2104 adapter (c) 2021 dushin.net v0.1.0"
- board text removed: "ESP32 CP2104 adapter (c) 2021 dushin.net v0.1.0-beta2"
