File: esp32-wroom-shield/esp32-wroom-shield.kicad_pcb (KiCad board)
At the start: 2 copper layers, 34.6 x 30.3 mm, 15 parts, among them J1 Conn_02x09_Odd_Even, J2 Conn_02x09_Odd_Even, SW1 RESET, SW2 PROG, U1 ESP32-WROOM-32

Commit message: Fixes to beta1 versions and added rws
Parts:
- added R2: 10k, Resistor_SMD:R_1206_3216Metric_Pad1.30x1.75mm_HandSolder, B.Cu at (147.6, 113.1)
- SW1, SW2: footprint Button_Switch_SMD:SW_SPST_B3U-1000P -> Button_Switch_SMD:SW_SPST_EVQPE1
- moved C4 2.21 mm to (150.0, 113.1)
- moved SW2 1.51 mm to (151.6, 112.2)
- moved SW1 1.49 mm to (134.3, 112.2)
- turned R1 to 270 degrees
- renumbered C4 to C3, C5 to C4, R2 to R3, R3 to R4
Connections:
- R1 pad 1: /VDD -> /EN
- R1 pad 2: /EN -> /VDD
Routing:
- net /IO0: track 16.9 -> 19.2 mm
Other:
- board text added: "ESP32 WROOM Shield (c) 2021 dushin.net v0.1.0-beta2"
- board text removed: "ESP32 WROOM Shield (c) 2021 dushin.net v0.1.0-beta1"

Commit message: Set version to v0.1.0
Other:
- board text added: "ESP32 WROOM Shield (c) 2021 dushin.net v0.1.0"
- board text removed: "ESP32 WROOM Shield (c) 2021 dushin.net v0.1.0-beta2"
